File: PCB/DAQBoardFront/DAQBoardFront.kicad_sch (KiCad schematic)
At the start: 35 parts, among them IC2 LMR51430YDDCR, J2 53375-0410, T1 AC1210-110-C, U5 TCAN1051VDRQ1

Commit message: Nearly functional DAQ boards with buck converters and SMD CAN modules
Parts:
- removed T1: AC1210-110-C, CFR-Footprint-Library:AC1210-110-C, symbol Device:Transformer_1P_1S
- added T1: (no value), CFR-Footprint-Library:AC1210-110-C, symbol CFR Library:AC1210-110-C
Connections:
- net CAN Hi: now also T1.4 (AB)
- net CAN Lo: now also T1.3 (SA)
- net ExtraAnalog: now also J1.4; no longer J1.1
- net FLSus: now also J1.2; no longer J1.3
- net FRSus: now also J1.1; no longer J1.4
- net SteeringAngle: now also J1.3; no longer J1.2
- net at R13.1, U5.7 (CANH): now also T1.1 (AA)
- net at R14.2, U5.6 (CANL): now also T1.2 (SB)
Changed lines of the file:
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@@
 	(wire
 		(pts
-			(xy 38.1 189.23) (xy 59.69 189.23)
-		)
-		(stroke
-			(width 0)
-			(type default)
-		)
-	)
-	(wire
-		(pts
 			(xy 55.88 102.87) (xy 55.88 105.41)
 		)
@@
 	(wire
 		(pts
-			(xy 27.94 48.26) (xy 36.83 48.26)
+			(xy 38.1 189.23) (xy 59.69 189.23)
 		)
 		(stroke
@@
 	(wire
 		(pts
-			(xy 246.38 78.74) (xy 246.38 76.2)
+			(xy 27.94 48.26) (xy 36.83 48.26)
 		)
 		(stroke
@@
 	(wire
 		(pts
-			(xy 38.1 186.69) (xy 59.69 186.69)
+			(xy 246.38 78.74) (xy 246.38 76.2)
 		)
 		(stroke
@@
 	(wire
 		(pts
+			(xy 38.1 186.69) (xy 59.69 186.69)
+		)
+		(stroke
+			(width 0)
+			(type default)
+		)
+	)
+	(wire
+		(pts
 			(xy 207.01 34.29) (xy 204.47 34.29)
 		)
@@
 	(wire
 		(pts
-			(xy 38.1 184.15) (xy 59.69 184.15)
-		)
-		(stroke
-			(width 0)
-			(type default)
-		)
-	)
-	(wire
-		(pts
 			(xy 90.17 38.1) (xy 95.25 38.1)
 		)
@@
 	(wire
 		(pts
+			(xy 38.1 184.15) (xy 59.69 184.15)
+		)
+		(stroke
+			(width 0)
+			(type default)
+		)
+	)
+	(wire
+		(pts
 			(xy 85.09 27.94) (xy 85.09 45.72)
 		)
@@
 	)
 	(label "FLSus"
-		(at 59.69 184.15 180)
+		(at 59.69 186.69 180)
 		(effects
 			(font
@@
 	)
 	(label "ExtraAnalog"
-		(at 59.69 189.23 180)
+		(at 59.69 181.61 180)
 		(effects
 			(font
@@
 	)
 	(label "SteeringAngle"
-		(at 59.69 186.69 180)
+		(at 59.69 184.15 180)
 		(effects
 			(font
@@
 	)
 	(label "FRSus"
-		(at 59.69 181.61 180)
+		(at 59.69 189.23 180)
 		(effects
 			(font
@@
 	)
 	(symbol
-		(lib_id "Device:Transformer_1P_1S")
-		(at 106.68 38.1 270)
-		(unit 1)
-		(body_style 1)
-		(exclude_from_sim no)
-		(in_bom yes)
-		(on_board yes)
-		(in_pos_files yes)
-		(dnp no)
-		(fields_autoplaced yes)
-		(property "Reference" "T1"
-			(at 113.03 36.8426 90)
-			(show_name no)
-			(do_not_autoplace no)
-			(effects
-				(font
-					(size 1.27 1.27)
-				)
-				(justify left)
-			)
-		)
-		(property "Value" "AC1210-110-C"
-			(at 113.03 39.3826 90)
-			(show_name no)
-			(do_not_autoplace no)
-			(effects
-				(font
-					(size 1.27 1.27)
-				)
-				(justify left)
-			)
-		)
-		(property "Footprint" "CFR-Footprint-Library:AC1210-110-C"
-			(at 106.68 38.1 0)
-			(hide yes)
-			(show_name no)
-			(do_not_autoplace no)
-			(effects
-				(font
-					(size 1.27 1.27)
-				)
-			)
-		)
-		(property "Datasheet" ""
-			(at 106.68 38.1 0)
-			(hide yes)
-			(show_name no)
-			(do_not_autoplace no)
-			(effects
-				(font
-					(size 1.27 1.27)
-				)
-			)
-		)
-		(property "Description" "Common-Mode Choke"
-			(at 106.68 38.1 0)
-			(hide yes)
-			(show_name no)
-			(do_not_autoplace no)
-			(effects
-				(font
-					(size 1.27 1.27)
-				)
-			)
-		)
-		(pin "3"
-		)
-		(pin "1"
-		)
-		(pin "4"
-		)
-		(pin "2"
-		)
-		(instances
-			(project "DAQBoardFront"
-				(path "/b8c14199-b7a8-42b0-9649-393d2e0c6b59"
-					(reference "T1")
-					(unit 1)
-				)
-			)
-		)
-	)
-	(symbol
 		(lib_id "Device:R")
 		(at 90.17 31.75 0)
@@
 					(unit 1)
 				)
+			)
+		)
+	)
+	(symbol
+		(lib_id "CFR Library:AC1210-110-C")
+		(at 101.6 27.94 90)
+		(mirror x)
+		(unit 1)
+		(body_style 1)
+		(exclude_from_sim no)
+		(in_bom yes)
+		(on_board yes)
+		(in_pos_files yes)
+		(dnp no)
+		(property "Reference" "T1"
+			(at 114.3 38.1 90)
+			(show_name no)
+			(do_not_autoplace no)
+			(effects
+				(font
+					(size 1.27 1.27)
+				)
+				(justify right)
+			)
+		)
+		(property "Value" ""
+			(at 101.6 27.94 0)
+			(show_name no)
+			(do_not_autoplace no)
+			(effects
+				(font
+					(size 1.27 1.27)
+				)
+			)
+		)
+		(property "Footprint" "CFR-Footprint-Library:AC1210-110-C"
+			(at 101.6 27.94 0)
+			(hide yes)
+			(show_name no)
+			(do_not_autoplace no)
+			(effects
+				(font
+					(size 1.27 1.27)
+				)
+			)
+		)
+		(property "Datasheet" ""
+			(at 101.6 27.94 0)
+			(hide yes)
+			(show_name no)
+			(do_not_autoplace no)
+			(effects
+				(font
+					(size 1.27 1.27)
+				)
+			)
+		)
+		(property "Description" "AC1210-110-C"
+			(at 101.6 27.94 0)
+			(hide yes)
+			(show_name no)
+			(do_not_autoplace no)
+			(effects
+				(font
+					(size 1.27 1.27)
+				)
+			)
+		)
+		(pin "1"
+		)
+		(pin "2"
+		)
+		(pin "3"
+		)
+		(pin "4"
+		)
+		(instances
+			(project "DAQBoardFront"
+				(path "/b8c14199-b7a8-42b0-9649-393d2e0c6b59"
+					(reference "T1")
+					(unit 1)
+				)
